File: rpi-hack-board.kicad_pcb (KiCad board)
At the start: 2 copper layers, 65 x 30 mm, 20 parts, among them J1 LOAD, J2 I2C_0, J3 I2C_1, J4 Raspberry_Pi_2_3, J5 PWR, J6 AP102, Q1 TIP120, U1 DS1307, X1 CRYSTAL

Commit message: Layout nearly done, interim check-in
Parts:
- added J7: SERIAL, Pin_Headers:Pin_Header_Straight_1x03_Pitch2.54mm, F.Cu at (145.7, 123.0)
- added J8: BREAKOUTS, Pin_Headers:Pin_Header_Straight_1x20_Pitch2.54mm, F.Cu at (108.4, 108.6)
- added REF**: Pin_Header_Straight_1x03_Pitch2.54mm, Pin_Headers:Pin_Header_Straight_1x03_Pitch2.54mm, F.Cu at (149.0, 112.2)
- added REF**: Pin_Header_Straight_1x03_Pitch2.54mm, Pin_Headers:Pin_Header_Straight_1x03_Pitch2.54mm, F.Cu at (126.1, 112.2)
- added REF**: Pin_Header_Straight_1x03_Pitch2.54mm, Pin_Headers:Pin_Header_Straight_1x03_Pitch2.54mm, F.Cu at (123.6, 112.2)
- added REF**: Pin_Header_Straight_1x03_Pitch2.54mm, Pin_Headers:Pin_Header_Straight_1x03_Pitch2.54mm, F.Cu at (121.1, 112.2)
- added REF**: Pin_Header_Straight_1x03_Pitch2.54mm, Pin_Headers:Pin_Header_Straight_1x03_Pitch2.54mm, F.Cu at (118.5, 112.2)
- added REF**: Pin_Header_Straight_1x03_Pitch2.54mm, Pin_Headers:Pin_Header_Straight_1x03_Pitch2.54mm, F.Cu at (116.0, 112.2)
- added REF**: Pin_Header_Straight_1x03_Pitch2.54mm, Pin_Headers:Pin_Header_Straight_1x03_Pitch2.54mm, F.Cu at (113.4, 112.2)
- added REF**: Pin_Header_Straight_1x03_Pitch2.54mm, Pin_Headers:Pin_Header_Straight_1x03_Pitch2.54mm, F.Cu at (146.5, 112.2)
- added REF**: Pin_Header_Straight_1x03_Pitch2.54mm, Pin_Headers:Pin_Header_Straight_1x03_Pitch2.54mm, F.Cu at (110.9, 112.2)
- added REF**: Pin_Header_Straight_1x03_Pitch2.54mm, Pin_Headers:Pin_Header_Straight_1x03_Pitch2.54mm, F.Cu at (143.9, 112.2)
- added REF**: Pin_Header_Straight_1x03_Pitch2.54mm, Pin_Headers:Pin_Header_Straight_1x03_Pitch2.54mm, F.Cu at (141.4, 112.2)
- added REF**: Pin_Header_Straight_1x03_Pitch2.54mm, Pin_Headers:Pin_Header_Straight_1x03_Pitch2.54mm, F.Cu at (138.8, 112.2)
- added REF**: Pin_Header_Straight_1x03_Pitch2.54mm, Pin_Headers:Pin_Header_Straight_1x03_Pitch2.54mm, F.Cu at (136.3, 112.2)
- added REF**: Pin_Header_Straight_1x03_Pitch2.54mm, Pin_Headers:Pin_Header_Straight_1x03_Pitch2.54mm, F.Cu at (133.8, 112.2)
- added REF**: Pin_Header_Straight_1x03_Pitch2.54mm, Pin_Headers:Pin_Header_Straight_1x03_Pitch2.54mm, F.Cu at (131.2, 112.2)
- added REF**: Pin_Header_Straight_1x03_Pitch2.54mm, Pin_Headers:Pin_Header_Straight_1x03_Pitch2.54mm, F.Cu at (128.7, 112.2)
- moved J6 15.1 mm to (162.5, 114.0)
- moved C1 9.13 mm to (151.5, 125.2)
- moved Q1 9.00 mm to (154.0, 118.0)
- moved R1 8.73 mm to (157.6, 117.3), turned to 270 degrees
- moved C2 1.17 mm to (102.5, 109.4), turned to 0 degrees
- moved X1 1.13 mm to (102.2, 121.9), turned to 180 degrees
- moved J5 0.79 mm to (162.5, 108.2)
- moved U1 0.79 mm to (103.6, 115.8)
- moved LED1 0.59 mm to (128.8, 127.0)
- moved J3 0.55 mm to (138.3, 120.4)
- moved J2 0.52 mm to (134.7, 120.4)
- moved J1 0.50 mm to (142.0, 123.0)
- moved BT1 0.22 mm to (115.7, 124.6)
- turned C3 to 180 degrees
Connections:
- net /DS_CO renamed /SCLK
- net /DS_DI renamed /MOSI
- J4 pad 1: Net-(J4-Pad1) -> /3.3V
- J4 pad 10: Net-(J4-Pad10) -> /RX
- J4 pad 11: Net-(J4-Pad11) -> /GPIO17
- J4 pad 13: Net-(J4-Pad13) -> /GPIO27
- J4 pad 15: Net-(J4-Pad15) -> /GPIO22
- J4 pad 21: Net-(J4-Pad21) -> /MISO
- J4 pad 24: Net-(J4-Pad24) -> /GPIO08
- J4 pad 26: Net-(J4-Pad26) -> /GPIO07
- J4 pad 31: Net-(J4-Pad31) -> /GPIO6
- J4 pad 32: Net-(J4-Pad32) -> /GPIO12
- J4 pad 8: Net-(J4-Pad8) -> /TX
Routing:
- net /SCL: track 0.00 -> 90.0 mm, vias 0 -> 2
- net /SDA: track 0.00 -> 71.2 mm, vias 0 -> 2
- net /TX: track 0.00 -> 54.4 mm
- net /RX: track 0.00 -> 48.7 mm, vias 0 -> 1
- net /WS2812: track 0.00 -> 36.0 mm
- net Net-(BT1-Pad1): track 0.00 -> 30.6 mm, vias 0 -> 2
- net GND: track 0.00 -> 15.2 mm, vias 0 -> 2
- net Net-(J1-Pad2): track 0.00 -> 13.5 mm
- net Net-(BT1-Pad2): track 0.00 -> 13.1 mm
- net /3.3V: track 0.00 -> 13.1 mm
- net /GPIO08: track 0.00 -> 10.1 mm
- net /GPIO07: track 0.00 -> 9.61 mm
- net /5V: track 0.00 -> 8.35 mm, vias 0 -> 1
- net /GPIO17: track 0.00 -> 8.33 mm
- net /GPIO22: track 0.00 -> 7.59 mm
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- added copper zone on F.Cu, net /5V
- added copper zone on B.Cu, net GND

Commit message: Getting closer, but still needs more work
Parts:
- J5: footprint Pin_Headers:Pin_Header_Straight_1x02_Pitch2.54mm -> Screw_Terminal_Vertical_1x02_Pitch2.54mm
- J6: value AP102 -> APA102
- moved J1 28.9 mm to (170.8, 125.5)
- moved R1 12.1 mm to (146.7, 122.6)
- moved J7 2.77 mm to (142.9, 123.1)
- moved C1 2.76 mm to (149.6, 127.2)
- moved Q1 2.19 mm to (156.2, 118.2)
- moved J6 0.76 mm to (161.8, 114.3)
- moved J5 0.70 mm to (161.8, 108.1)
- moved J3 0.56 mm to (138.9, 120.5)
- moved J2 0.15 mm to (134.8, 120.5)
Routing:
- net Net-(J1-Pad2): track 13.5 -> 0.00 mm
- net (no net): track 3.70 -> 0.00 mm
- net /TX: track 54.4 -> 55.5 mm

Commit message: SOOOOO CLOSE!
Parts:
- J1: footprint Pin_Headers:Pin_Header_Straight_1x03_Pitch2.54mm -> mayhem-footprints:Screw_Terminal_Vertical_1x02_Pitch2.54mm
- J5: footprint Screw_Terminal_Vertical_1x02_Pitch2.54mm -> mayhem-footprints:Screw_Terminal_Vertical_1x02_Pitch2.54mm
- moved J1 14.2 mm to (156.7, 126.8), turned to 270 degrees
- moved R1 14.1 mm to (155.8, 111.8), turned to 180 degrees
- moved C1 7.98 mm to (141.8, 125.5)
- moved J7 7.56 mm to (150.5, 123.0)
- moved Q1 2.52 mm to (156.2, 120.7)
- moved J3 0.74 mm to (138.2, 120.5)
- moved J2 0.24 mm to (134.6, 120.5)
Connections:
- J4 pad 29: /LOAD_DRV -> Net-(J4-Pad29)
- J4 pad 37: Net-(J4-Pad37) -> /LOAD_DRV
Routing:
- net /MOSI: track 4.95 -> 65.7 mm
- net /SCLK: track 4.86 -> 44.0 mm, vias 0 -> 1
- net /WS2812: track 36.0 -> 0.00 mm
- net /RX: track 48.2 -> 66.7 mm, vias 1 -> 0
- net Net-(Q1-Pad1): track 0.00 -> 11.6 mm, vias 0 -> 1
- net Net-(J1-Pad2): track 0.00 -> 10.3 mm
- net /LOAD_DRV: track 0.00 -> 9.01 mm
- net /5V: track 8.35 -> 3.26 mm, vias 1 -> 0
- net GND: track 15.2 -> 12.1 mm, vias 2 -> 1

Commit message: Layout is complete, remaining connections are not needed!
Connections:
- J4 pad 33: /WS2812 -> Net-(J4-Pad33)
- J4 pad 40: Net-(J4-Pad40) -> /WS2812
Routing:
- net /WS2812: track 0.00 -> 47.0 mm, vias 0 -> 2
- net Net-(BT1-Pad1): track 30.6 -> 7.55 mm, vias 2 -> 0
- net /SCLK: track 44.0 -> 50.1 mm
- net GND: track 12.1 -> 16.1 mm, vias 1 -> 2
- net /MOSI: track 65.7 -> 66.5 mm, vias 0 -> 2
- net /RX: vias 0 -> 2
